File: esp32-mini.kicad_sch (KiCad schematic)
At the start: 23 parts, among them J1 Conn_01x11, J3 USB_C_Receptacle, SW1 SMD_4.6x2.8mm_h2.5mm, SW2 SMD_4.6x2.8mm_h2.5mm, U1 ESP32-C3-MINI-1-N4, U6 AMS1117-3.3

Commit message: update readme.md
Other:
- note removed: "Geo_Pro Lite"
Changed lines of the file:
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@@
-		)
-	)
-	(text "Geo_Pro Lite"
-		(exclude_from_sim no)
-		(at 195.834 189.738 0)
-		(effects
-			(font
-				(size 1.56 1.56)
-				(thickness 0.254)
-				(bold yes)
-			)
 		)
 	)
