File: esp32-mini.kicad_sch (KiCad schematic)
At the start: 23 parts, among them J1 Conn_01x11, J3 USB_C_Receptacle, SW1 SMD_4.6x2.8mm_h2.5mm, SW2 SMD_4.6x2.8mm_h2.5mm, U1 ESP32-C3-MINI-1-N4, U6 AMS1117-3.3

Commit message: minor fixes
Parts:
- removed C3, C4: 0.1uF, PCM_SparkFun-Capacitor:C_0402_1005Metric, symbol PCM_SparkFun-Capacitor:0.1uF_0402_16V_10%
- added C10, C11: 0.1uF, PCM_SparkFun-Capacitor:C_0402_1005Metric, symbol PCM_SparkFun-Capacitor:0.1uF_0402_16V_10%
- C15: value 1.0uF -> 10uF; footprint PCM_SparkFun-Capacitor:C_0402_1005Metric -> PCM_SparkFun-Capacitor:C_0603_1608Metric; symbol PCM_SparkFun-Capacitor:1.0uF_0402_16V_10% -> PCM_SparkFun-Capacitor:10uF_0603_6.3V_20%; Tolerance 10% -> 20%; Voltage 16V -> 6.3V
Connections:
- net GND: now also C10.2, C11.2
- net chip_pu: now also C11.1
- net I01 renamed IO1
- net I02 renamed IO2
- net I03 renamed IO3
- net I04 renamed IO4
- net Io0 renamed IO0
- net gpio9 renamed IO9
- net IO9: now also C10.1
