File: esp32-mini.kicad_pcb (KiCad board)
At the start: 2 copper layers, 23 parts, among them J1 Conn_01x11, J3 USB_C_Receptacle, SW1 SMD_4.6x2.8mm_h2.5mm, SW2 SMD_4.6x2.8mm_h2.5mm, U1 ESP32-C3-MINI-1-N4, U6 AMS1117-3.3

Commit message: update schematic and pcb layout
Parts:
- moved C5 16.4 mm to (75.0, 78.5), turned to 90 degrees
- moved C1 2.56 mm to (72.0, 62.5)
Routing:
- net GND: track 0.00 -> 173.4 mm, vias 0 -> 2
- net chip_pu: track 0.00 -> 72.4 mm, vias 0 -> 5
- net 3V3: track 0.00 -> 58.2 mm, vias 0 -> 4
- net gpio9: track 0.00 -> 56.2 mm, vias 0 -> 3
- net Net-(D1-A): track 0.00 -> 53.6 mm, vias 0 -> 2
- net TxD0: track 0.00 -> 31.3 mm, vias 0 -> 2
- net Net-(J3-CC1): track 0.00 -> 31.1 mm, vias 0 -> 2
- net Net-(J3-CC2): track 0.00 -> 30.9 mm, vias 0 -> 2
- net I03: track 0.00 -> 25.3 mm, vias 0 -> 2
- net I02: track 0.00 -> 24.4 mm, vias 0 -> 1
- net IO10: track 0.00 -> 23.0 mm, vias 0 -> 1
- net RxD0: track 0.00 -> 21.2 mm, vias 0 -> 1
- net Io0: track 0.00 -> 19.6 mm, vias 0 -> 1
- net D-: track 0.00 -> 18.2 mm, vias 0 -> 2
- net 5V: track 0.00 -> 17.3 mm, vias 0 -> 2
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- added copper zone on F.Cu, net GND
Other:
- board outline added: 37.5 x 35.5 mm
- board text added: "Io0 Io1 Io2 Io3 Io4 Io5 Io6 Io8 Io10 Rx Tx"
