File: esp32-mini.kicad_pcb (KiCad board)
At the start: 2 copper layers, 37.5 x 35.5 mm, 23 parts, among them J1 Conn_01x11, J3 USB_C_Receptacle, SW1 SMD_4.6x2.8mm_h2.5mm, SW2 SMD_4.6x2.8mm_h2.5mm, U1 ESP32-C3-MINI-1-N4, U6 AMS1117-3.3

Commit message: minor fixes
Parts:
- C15: value 1.0uF -> 10uF
Connections:
- net I01 renamed IO1
- net I02 renamed IO2
- net I03 renamed IO3
- net I04 renamed IO4
- net Io0 renamed IO0
- net gpio9 renamed IO9
- U6 pad 4: GND -> 3V3
Other:
- board text added: "IO0 IO1 IO2 IO3 IO4 IO5 IO6 IO8 IO10 Rx Tx"
- board text removed: "Io0 Io1 Io2 Io3 Io4 Io5 Io6 Io8 Io10 Rx Tx"
Changed lines of the file:
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@@
 	(net 1 "GND")
 	(net 2 "3V3")
-	(net 3 "gpio9")
+	(net 3 "IO9")
 	(net 4 "chip_pu")
 	(net 5 "5V")
@@
 	(net 8 "TxD0")
 	(net 9 "IO5")
-	(net 10 "Io0")
+	(net 10 "IO0")
 	(net 11 "RxD0")
 	(net 12 "IO10")
-	(net 13 "I04")
-	(net 14 "I01")
+	(net 13 "IO4")
+	(net 14 "IO1")
 	(net 15 "IO6")
-	(net 16 "I02")
+	(net 16 "IO2")
 	(net 17 "IO8")
-	(net 18 "I03")
+	(net 18 "IO3")
 	(net 19 "Net-(J3-CC1)")
 	(net 20 "unconnected-(J3-NC-PadNC1)")
@@
 			(layers "F.Cu" "F.Mask" "F.Paste")
 			(roundrect_rratio 0.075)
-			(net 1 "GND")
-			(pinfunction "ADJ")
-			(pintype "power_in")
+			(net 2 "3V3")
+			(pinfunction "VOUT")
+			(pintype "output")
 			(solder_mask_margin 0.102)
 		)
@@
 			(size 0.8 0.4)
 			(layers "F.Cu" "F.Mask" "F.Paste")
-			(net 16 "I02")
+			(net 16 "IO2")
 			(pinfunction "IO2")
 			(pintype "bidirectional")
@@
 			(size 0.8 0.4)
 			(layers "F.Cu" "F.Mask" "F.Paste")
-			(net 18 "I03")
+			(net 18 "IO3")
 			(pinfunction "IO3")
 			(pintype "bidirectional")
@@
 			(size 0.4 0.8)
 			(layers "F.Cu" "F.Mask" "F.Paste")
-			(net 10 "Io0")
+			(net 10 "IO0")
 			(pinfunction "IO0")
 			(pintype "bidirectional")
@@
 			(size 0.4 0.8)
 			(layers "F.Cu" "F.Mask" "F.Paste")
-			(net 14 "I01")
+			(net 14 "IO1")
 			(pinfunction "IO1")
 			(pintype "bidirectional")
@@
 			(size 0.4 0.8)
 			(layers "F.Cu" "F.Mask" "F.Paste")
-			(net 13 "I04")
+			(net 13 "IO4")
 			(pinfunction "IO4")
 			(pintype "bidirectional")
@@
 			(size 0.4 0.8)
 			(layers "F.Cu" "F.Mask" "F.Paste")
-			(net 3 "gpio9")
+			(net 3 "IO9")
 			(pinfunction "IO9")
 			(pintype "bidirectional")
@@
 			(size 0.9 1)
 			(layers "F.Cu" "F.Mask" "F.Paste")
-			(net 3 "gpio9")
+			(net 3 "IO9")
 			(pinfunction "2")
 			(pintype "passive")
@@
 			(size 0.9 1)
 			(layers "F.Cu" "F.Mask" "F.Paste")
-			(net 3 "gpio9")
+			(net 3 "IO9")
 			(pinfunction "2")
 			(pintype "passive")
@@
 			)
 		)
-		(property "Value" "1.0uF"
-			(at 0 1.16 0)
+		(property "Value" "10uF"
+			(at 0 1.43 0)
 			(layer "F.Fab")
 			(effects
@@
 			(layers "F.Cu" "F.Mask" "F.Paste")
 			(roundrect_rratio 0.25)
-			(net 3 "gpio9")
+			(net 3 "IO9")
 			(pintype "passive")
 		)
@@
 			(keep_end_layers yes)
 			(zone_layer_connections)
-			(net 10 "Io0")
+			(net 10 "IO0")
 			(pinfunction "Pin_1")
 			(pintype "passive")
@@
 			(keep_end_layers yes)
 			(zone_layer_connections)
-			(net 14 "I01")
+			(net 14 "IO1")
 			(pinfunction "Pin_2")
 			(pintype "passive")
@@
 			(keep_end_layers yes)
 			(zone_layer_connections)
-			(net 16 "I02")
+			(net 16 "IO2")
 			(pinfunction "Pin_3")
 			(pintype "passive")
@@
 			(keep_end_layers yes)
 			(zone_layer_connections)
-			(net 18 "I03")
+			(net 18 "IO3")
 			(pinfunction "Pin_4")
 			(pintype "passive")
@@
 			(keep_end_layers yes)
 			(zone_layer_connections)
-			(net 13 "I04")
+			(net 13 "IO4")
 			(pinfunction "Pin_5")
 			(pintype "passive")
@@
 			(layers "F.Cu" "F.Mask" "F.Paste")
 			(roundrect_rratio 0.25)
-			(net 3 "gpio9")
+			(net 3 "IO9")
 			(pintype "passive")
 		)
@@
 			)
 		)
-		(property "Voltage" "6.3V"
+		(property "Voltage" "10V"
 			(at 0 0 90)
 			(unlocked yes)
@@
 		(layer "Edge.Cuts")
 	)
-	(gr_text "Io0 Io1 Io2 Io3 Io4 Io5 Io6 Io8 Io10 Rx Tx"
+	(gr_text "IO0 IO1 IO2 IO3 IO4 IO5 IO6 IO8 IO10 Rx Tx"
 		(at 70 87.5 0)
 		(layer "F.SilkS")
